Commit message: change urdf file to urdf of sff01

File: diffdrive/diff_description/urdf/robot_core.xacro (robot description, xacro)
@@ -2,18 +2,18 @@
 <robot xmlns:xacro="http://www.ros.org/wiki/xacro" >
     <xacro:include filename="inertial_macros.xacro"/>
-    <xacro:property name="chassis_length" value="0.20"/>
+    <xacro:property name="chassis_length" value="0.725"/>
     <xacro:property name="chassis_width" value="0.15"/>
     <xacro:property name="chassis_height" value="0.043"/>
     <xacro:property name="chassis_mass" value="0.24"/>
-    <xacro:property name="wheel_radius" value="0.033"/>
+    <xacro:property name="wheel_radius" value="0.0855"/>
     <xacro:property name="wheel_thickness" value="0.024"/>
     <xacro:property name="wheel_mass" value="0.05"/>
     <xacro:property name="wheel_offset_x" value="0.035"/>
-    <xacro:property name="wheel_offset_y" value="0.089"/>
+    <xacro:property name="wheel_offset_y" value="0.2355"/>
     <xacro:property name="wheel_offset_z" value="0.0215"/>
-    <xacro:property name="caster_wheel_radius" value="0.0125"/>
+    <xacro:property name="caster_wheel_radius" value="0.05"/>
     <xacro:property name="caster_wheel_mass" value="0.01"/>
-    <xacro:property name="caster_wheel_offset_x" value="0.18145"/>
-    <xacro:property name="caster_wheel_offset_z" value="0.03517"/>
+    <xacro:property name="caster_wheel_offset_x" value="0.70645"/>
+    <xacro:property name="caster_wheel_offset_z" value="0.057"/>
     <material name="white">
         <color rgba="1 1 1 1" />

Commit message: spaw robot into world and fix control lag

File: diffdrive/diff_description/urdf/robot_core.xacro (robot description, xacro)
@@ -3,9 +3,9 @@
     <xacro:include filename="inertial_macros.xacro"/>
     <xacro:property name="chassis_length" value="0.725"/>
-    <xacro:property name="chassis_width" value="0.15"/>
+    <xacro:property name="chassis_width" value="0.3"/>
     <xacro:property name="chassis_height" value="0.043"/>
     <xacro:property name="chassis_mass" value="0.24"/>
     <xacro:property name="wheel_radius" value="0.0855"/>
-    <xacro:property name="wheel_thickness" value="0.024"/>
+    <xacro:property name="wheel_thickness" value="0.08"/>
     <xacro:property name="wheel_mass" value="0.05"/>
     <xacro:property name="wheel_offset_x" value="0.035"/>
